File: hardware/kicad/_autosave-vuulgaris.kicad_pcb (KiCad board)
At the start: 2 copper layers, 284.3 x 125 mm, 69 parts, among them J1 TFPUSH, J10 PJ-603_C41409498, J11 TYPE-C-31-M-12, J2 PJ-376, J3 PJ-376, J4 PJ-376, J5 PJ-376, J7 PJ-603_C41409498, J8 PJ-603_C41409498, J9 PJ-603_C41409498, SW4 CPG151101S03, SW5 CPG151101S03, SW6 CPG151101S03, SW7 CPG151101S03, U1 ES_DAISY_PATCH_SM_REV1, U3 MCP23017-E_SO, U4 MCP23017-E_SO, U5 AMS1117-3.3, U6 AMS1117-3.3, U7 DKM10E-12

Commit message: hardware: Daisy to the bottom edge for the exposed micro-USB
The micro-USB is being exposed after all, so U1 has to sit on a board edge
again. The bottom is the only one with a free 68mm span: the top edge is jacks
end to end, the right is the power stage, the left is the MX cluster. U1 lands at
x[86,154] y[85,125], hard against the edge, still on B.Cu.

J1 turns 180 -> 0 with it. At 180 the mouth faced +y, which is now straight into
the Daisy; at 0 the mouth faces -y so the card ejects upward into open board
while the contacts face down toward the D header. SDIO drops to about 9mm and the
card path is unobstructed. Safe as a text edit because its pads are rectangles
and a 180 turn preserves their width and height.

I corrupted the board file getting here and restored it from 47ecdb0. The
rotation script located the footprint with str.find and had no guard for find
returning -1 on the following footprint, so instead of one block it rewrote every
angle from J1 to the end of the file: U1 came back F.Cu at -90 hanging 14mm off
the bottom edge, and U6 and FB2 were spun too. place.py already contains a
brace-matching block reader written for exactly this; the redo uses it and then
diffs the parsed footprint table before and after, refusing to write unless the
changed set is exactly {J1}. Any future single-footprint edit should do the same
-- the check costs four lines and it is the difference between a bad edit that
announces itself and one that does not.

Still unknown, and now blocking: which edge of the module the micro-USB exits.
The carrier footprint has pin groups on all four sides, so it cannot be inferred
from the file.
Parts:
- F1: moved to B.Cu
- J1, J11, U1: moved to F.Cu
- moved J1 178.6 mm to (374.4, 86.6), turned to -90 degrees
- moved U1 145.1 mm to (363.8, 136.1), turned to -90 degrees
- moved L2 53.5 mm to (296.0, 140.0)
- moved R20 53.3 mm to (286.7, 122.4)
- moved R21 53.3 mm to (286.7, 128.4)
- moved U7 53.0 mm to (318.9, 126.0)
- moved C36 52.8 mm to (304.1, 144.1)
- moved C37 52.8 mm to (304.1, 154.1)
- moved C38 52.8 mm to (304.1, 149.1)
- moved C39 52.8 mm to (304.1, 159.1)
- moved D1 52.7 mm to (317.2, 149.8)
- moved D2 52.7 mm to (317.2, 159.8)
- moved R24 52.7 mm to (313.2, 149.8)
- moved R25 52.7 mm to (313.2, 159.8)
- moved C32 48.6 mm to (300.6, 116.4)
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