File: hardware/kicad/vuulgaris.kicad_sch (KiCad schematic)
At the start: 81 parts, among them J1 TFPUSH, J10 PJ-603_C41409498, J11 TYPE-C-31-M-12, J2 PJ-376, J3 PJ-376, J4 PJ-376, J5 PJ-376, J7 PJ-603_C41409498, J8 PJ-603_C41409498, J9 PJ-603_C41409498, SW4 CPG151101S03, SW5 CPG151101S03, SW6 CPG151101S03, SW7 CPG151101S03, U1 ES_DAISY_PATCH_SM_REV1, U10 DG419DY-T1-E3, U11 DG419DY-T1-E3, U3 MCP23017-E_SO, U4 MCP23017-E_SO, U5 AMS1117-3.3, U6 AMS1117-3.3, U7 DKM10E-12, U8 DG419DY-T1-E3, U9 DG419DY-T1-E3

Commit message: hardware: SW1/SW2 back to mechanical -- Dailywell DW3, footprint from the drawing
Reverts the DG419 analog switches. U8-U11 and their eight decoupling caps are
gone, U4 GPB3/GPB4 are spare again, and SW1/SW2 are mechanical DPDT toggles.

The part is a Dailywell 2MD1T1B1M2QES, DPDT ON-ON, PC pin -- Thonk sell it as
DW3. It is the Eurorack DIY standard, used by Music Thing and Zlob among others,
and Thonk's own note is what settles the question that blocked this all
afternoon: soldered into a PCB these "sit at a height that matches box-style
3.5mm sockets and PCB mounting pots", which is exactly this board's geometry.
That is the reach problem answered by the part rather than worked around.

The footprint is drawn from the manufacturer drawing 2MDP0428 rev C, not from
memory. Fetched the PDF, rendered it, and read the P.C. MOUNTING detail directly:
two columns 5.08mm apart, three pins per column at 2.54mm, 1.09mm holes. Panel
hole 4.95mm, bushing 10-48 UNS-2A x 5.59mm long. The drawing also confirms the
contact table -- POS.1 makes 2-3 and 5-6, POS.3 makes 2-1 and 5-4, so pins 2 and
5 are the commons and the throws are 1/3 and 4/6. design-state predicted exactly
that and told us to verify it rather than assume; now it is verified, and the
note about checking with a meter applies only to substitutes.

The faceplate opening changes with it. It had been a 9 x 20mm vertical SLOT,
which suited a slide actuator; this switch needs a ROUND 4.95mm bushing hole.
switch_w/h stay as the layout footprint the switch occupies in the row so nothing
reflows, and switch_hole_d_mm is what actually gets cut. The stale "switch slots
vertical" check is replaced by one that asserts the hole fits its column.

Pins stay unwired until Bergman's circuit lands, as with RV1-RV4.

217/217 netcheck, faceplate clean, all 20 panel parts on their holes, no
overlaps, Gerbers clean. Board needs F8 to pick up SW1/SW2.
Parts:
- removed C40, C41, C42, C43, C44, C45, C46, C47: CL05B104KO5NNNC, vuulgaris:C0402, symbol vuulgaris:CL05B104KO5NNNC
- removed U10, U11, U8, U9: DG419DY-T1-E3, vuulgaris:SOIC-8_L4.9-W3.9-P1.27-LS6.0-BL, symbol vuulgaris:DG419DY-T1-E3
- added SW1, SW2: SW_DPDT_x2, vuulgaris:SW-TH_DW3_DPDT_2MD1T1B1M2QES, symbol vuulgaris:SW_DPDT_x2
Connections:
- net MODE_SEL: no longer names the net of U4.4 (GPB3)
- net SRC_SEL: no longer names the net of U4.5 (GPB4)
- no-connect marks 123 -> 125

Commit message: hardware: stereo BBD delay block, built from the SSI2100 reference circuit
92 new parts. Schematic verifies 440/440 with nothing unintended, up from
217/217. Everything is placed except the three parts Dylan solders himself: the
two SSI2100s and the SSI2164 VCA.

Per channel, straight from Figure 1 -- 3-pole anti-alias filter in at 15kHz, the
100R/1nF network that stabilises the sample-and-hold input, the BBD, a 5k trim
balancing the two source-follower outputs into a 49.9k load, and a 4-pole
reconstruction filter out. The V_DCB divider is shared: 18.2k/32.4k off +5V gives
the 3.20V the SIGNAL IN pin requires, and it is a DC reference so both channels
can hang off it.

Wet/dry is a VCA rather than a pot, because the panel is full and this way it
recalls with the patch. Two of the SSI2164's four cells set wet level while dry
is summed into the same virtual earth, so one op-amp section per channel does the
current-to-voltage conversion AND the mix. Control comes from an MCP4728 quad DAC
on the existing I2C bus -- no new Daisy pins, and two DAC channels spare.

The clock arrangement is left as an experiment, as asked. The Daisy drives CLK_A
and CLK_B out to two test points; two more feed the BBDs. Jumper A to both for a
single shared clock (phase-locked stereo, no intermodulation) or A to L and B to
R for independent clocks. Bypass is a 3-pin header per channel: send, return
downstream, and the mix output, so the board works with the whole block
unpopulated.

Two supporting changes were needed:

mksch.py now reads per-ref values from tools/values.json. Until now Value was
always the symbol name, which is survivable for an MCU and useless for a filter,
where the value IS the design -- a schematic reading "CC0603JRX7R8BB104" instead
of "470pF" cannot be built from.

TL074 and the trim pot got flat single-unit symbols in the project library.
KiCad's TL074 is multi-unit and mksch.py emits exactly one instance per
reference, and KiCad's R_Trim has only two terminals where F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
Parts:
- added C40, C48, C61: 4.7uF, vuulgaris:C0805, symbol vuulgaris:CC0603JRX7R8BB104
- added C41, C46, C54, C59: 3.3uF, vuulgaris:C0805, symbol vuulgaris:CC0603JRX7R8BB104
- added C42, C43, C51, C55, C56, C64: 470pF, vuulgaris:C0603, symbol vuulgaris:CC0603JRX7R8BB104
- added C44, C57: 47pF, vuulgaris:C0603, symbol vuulgaris:CC0603JRX7R8BB104
- added C45, C58: 1nF, vuulgaris:C0603, symbol vuulgaris:CC0603JRX7R8BB104
- added C47, C60, C67, C68, C69, C70, C71, C72, C73, C74: 100nF, vuulgaris:C0603, symbol vuulgaris:CC0603JRX7R8BB104
- added C49, C62: 330pF, vuulgaris:C0603, symbol vuulgaris:CC0603JRX7R8BB104
- added C50, C63: 390pF, vuulgaris:C0603, symbol vuulgaris:CC0603JRX7R8BB104
- added C52, C65: 33pF, vuulgaris:C0603, symbol vuulgaris:CC0603JRX7R8BB104
- added C53, C66: 100pF, vuulgaris:C0603, symbol vuulgaris:CC0603JRX7R8BB104
- added J12, J13: BYPASS, vuulgaris:PinHeader_1x03_P2.54mm_Vertical, symbol vuulgaris:Conn_01x03
- added R26: 18.2k, vuulgaris:R0603, symbol vuulgaris:RT0603BRD075K1L
- added R27: 32.4k, vuulgaris:R0603, symbol vuulgaris:RT0603BRD075K1L
- added R28, R32, R40, R41, R42, R43, R44, R48, R56, R57, R58, R59: 100k, vuulgaris:R0603, symbol vuulgaris:RT0603BRD075K1L
- added R29, R45: 47k, vuulgaris:R0603, symbol vuulgaris:RT0603BRD075K1L
- added R30, R46: 56k, vuulgaris:R0603, symbol vuulgaris:RT0603BRD075K1L
- added R31, R38, R47, R54: 33k, vuulgaris:R0603, symbol vuulgaris:RT0603BRD075K1L
- added R33, R49: 100R, vuulgaris:R0603, symbol vuulgaris:RT0603BRD075K1L
- added R34, R50: 49.9k, vuulgaris:R0603, symbol vuulgaris:RT0603BRD075K1L
- added R35, R51: 43k, vuulgaris:R0603, symbol vuulgaris:RT0603BRD075K1L
- added R36, R37, R52, R53: 39k, vuulgaris:R0603, symbol vuulgaris:RT0603BRD075K1L
- added R39, R55: 120k, vuulgaris:R0603, symbol vuulgaris:RT0603BRD075K1L
- added RV5, RV6: 5k, vuulgaris:Potentiometer_Bourns_3266W_Vertical, symbol vuulgaris:TRIMPOT_3T
- added TP1, TP10, TP2, TP3, TP4, TP5, TP6, TP7, TP8, TP9: TP, vuulgaris:TestPoint_Pad_D1.5mm, symbol vuulgaris:TestPoint
- added U10, U11: SSI2100, vuulgaris:SOIC-8_L4.9-W3.9-P1.27-LS6.0-BL, symbol vuulgaris:SSI2100
- added U12: SSI2164, vuulgaris:SOIC-16_3.9x9.9mm_P1.27mm, symbol vuulgaris:SSI2164
- added U13: MCP4728, vuulgaris:MSOP-10_3x3mm_P0.5mm, symbol vuulgaris:MCP4728
- added U8, U9: TL074, vuulgaris:SOIC-14_3.9x8.7mm_P1.27mm, symbol vuulgaris:TL074_FLAT
Connections:
- net GND: now also C40.2, C42.2, C43.2, C45.2, C46.2, C47.2, C49.2, C50.2, C51.2, C55.2, C56.2, C58.2, C59.2, C60.2, C62.2, C63.2, C64.2, C67.2, C68.2, C69.2, C70.2, C71.2, C72.2, C73.2, C74.2, R27.2, R28.2, R34.2, R44.2, R50.2, U10.1 (GND), U10.2 (GCAP), U11.1 (GND), U11.2 (GCAP), U12.1 (MODE), U12.8 (GND), U13.10 (VSS), U13.4 (~{LDAC}), U8.12 (IN_D+), U8.5 (IN_B+), U9.10 (IN_C+), U9.12 (IN_D+), U9.3 (IN_A+), U9.5 (IN_B+)
- net I2C_SCL: now also U13.2 (SCL)
- net I2C_SDA: now also U13.3 (SDA)
- net NEG12V: now also C68.1, C70.1, C72.1, U12.9 (V-), U8.11 (V-), U9.11 (V-)
- net P3V3_DAISY: now also C73.1, U13.1 (VDD)
- net P5V: now also C47.1, C60.1, C74.1, R26.1, TP10.1, U10.7 (V+), U11.7 (V+)
- net POS12V: now also C67.1, C69.1, C71.1, U12.16 (V+), U8.4 (V+), U9.4 (V+)
- net CLK_A: now reaches U1.D3 (SDMMC_D2)
- net CLK_A: now also TP7.1
- net CLK_B: now reaches U1.D4 (SDMMC_D1)
- net CLK_B: now also TP8.1
- new net BBD_L_CLK: TP3.1, U10.8 (CLK_IN)
- new net BBD_L_CV: R43.2, U12.3 (VC1)
- new net BBD_L_F1: C41.2, R29.1
- new net BBD_L_F2: C42.1, R29.2, R30.1
- new net BBD_L_F3: C43.1, R30.2, R31.1, R32.1
- new net BBD_L_FIN: C44.1, R31.2, U8.2 (IN_A-)
- new net BBD_L_FOUT: C44.2, R32.2, R33.1, U8.1 (OUT_A)
- new net BBD_L_MIX: C53.2, J12.3 (Pin_3), R42.2, U9.1 (OUT_A)
- new net BBD_L_O1: RV5.1, U10.6 (SIG_OUT_1)
- new net BBD_L_O2: RV5.3, U10.5 (SIG_OUT_2)
- new net BBD_L_OW: C48.1, R34.1, RV5.2 (WIPER)
- new net BBD_L_RA: C48.2, R35.1
- new net BBD_L_RB: C49.1, R35.2, R36.1
- new net BBD_L_RC: C50.1, R36.2, R37.1
- new net BBD_L_RD: C51.1, R37.2, R38.1, R39.1
- new net BBD_L_RET: J12.2 (Pin_2)
- new net BBD_L_RIN: C52.1, R38.2, U8.6 (IN_B-)
- new net BBD_L_SEND: C41.1, J12.1 (Pin_1), R28.1, R41.1
- new net BBD_L_SIG: C45.1, R33.2, TP1.1, U10.3 (SIGNAL_IN)
- new net BBD_L_SUM: C53.1, R41.2, R42.1, U12.4 (I_OUT1), U9.2 (IN_A-)
- new net BBD_L_VIN: R40.2, U12.2 (I_IN1)
- new net BBD_L_VTB: C46.1, U10.4 (VTBIAS)
- new net BBD_L_WET: C52.2, R39.2, R40.1, TP2.1, U8.7 (OUT_B)
- new net BBD_R_CLK: TP6.1, U11.8 (CLK_IN)
- new net BBD_R_CV: R59.2, U12.6 (VC2)
- new net BBD_R_F1: C54.2, R45.1
- new net BBD_R_F2: C55.1, R45.2, R46.1
- new net BBD_R_F3: C56.1, R46.2, R47.1, R48.1
- new net BBD_R_FIN: C57.1, R47.2, U8.9 (IN_C-)
- new net BBD_R_FOUT: C57.2, R48.2, R49.1, U8.8 (OUT_C)
- new net BBD_R_MIX: C66.2, J13.3 (Pin_3), R58.2, U9.7 (OUT_B)
- new net BBD_R_O1: RV6.1, U11.6 (SIG_OUT_1)
- new net BBD_R_O2: RV6.3, U11.5 (SIG_OUT_2)
- new net BBD_R_OW: C61.1, R50.1, RV6.2 (WIPER)
- new net BBD_R_RA: C61.2, R51.1
- new net BBD_R_RB: C62.1, R51.2, R52.1
- new net BBD_R_RC: C63.1, R52.2, R53.1
- new net BBD_R_RD: C64.1, R53.2, R54.1, R55.1
- new net BBD_R_RET: J13.2 (Pin_2)
- new net BBD_R_RIN: C65.1, R54.2, U8.13 (IN_D-)
- new net BBD_R_SEND: C54.1, J13.1 (Pin_1), R44.1, R57.1
- new net BBD_R_SIG: C58.1, R49.2, TP4.1, U11.3 (SIGNAL_IN)
- new net BBD_R_SUM: C66.1, R57.2, R58.1, U12.5 (I_OUT2), U9.6 (IN_B-)
- new net BBD_R_VIN: R56.2, U12.7 (I_IN2)
- new net BBD_R_VTB: C59.1, U11.4 (VTBIAS)
- new net BBD_R_WET: C65.2, R55.2, R56.1, TP5.1, U8.14 (OUT_D)
- new net DAC_L: R43.1, U13.6 (VOUTA)
- new net DAC_R: R59.1, U13.7 (VOUTB)
- new net U9_C_N: U9.8 (OUT_C), U9.9 (IN_C-)
- new net U9_D_N: U9.13 (IN_D-), U9.14 (OUT_D)
- new net VDCB: C40.1, R26.2, R27.1, TP9.1, U8.10 (IN_C+), U8.3 (IN_A+)
- no-connect marks 125 -> 132

Commit message: hardware: rebuild the wet/dry VCA from the SSI2164 datasheet
The BBD signal path was transcribed from the SSI2100's Figure 1 and Dylan
verified it node by node. The VCA mix in that same commit was not from any
reference -- I designed it from general principles about current-mode VCAs and
let the commit message imply the whole block came from the datasheet. It did not,
and the invented half was wrong in most of its numbers.

What the datasheet says, and what I had:

  * control port input impedance is 9-11k, NOT high impedance. Feeding it through
    a 100k series resistor made a 10:1 divider, so the DAC's full 0-3.3V swing
    bought roughly 9dB of range out of an available 100dB.
  * gain constant is -33mV/dB and unity gain is at VC = 0.0V, positive
    attenuating. None of that was scaled for.
  * RIN should be 20k -- I used 100k, the noisiest end of the permitted range.
  * MODE is a current-set pin needing a resistor to V-, not a short to ground.
    Class A at +/-12V with IM = 1mA gives 5.6k, and the datasheet's own 9V ->
    3.9k example confirms the formula.
  * the control port wants a series 10uF for control feedthrough. Absent.

Replaced with Figure 10, the 0-5V exponential control circuit: an inverting
summing amp (100k in, 100k feedback, 100pF, 270k offset from -12V) driving the
control port through a 10uF cap, with a PNP clamp referenced to +2.7V from a
3k:10k divider limiting attenuation to 100dB. U9's C and D sections, which had
been tied off as followers, now do this work.

Also recorded in docs/bbd-ssi2100.md, including a table of exactly what the first
attempt got wrong, so the failure is legible rather than quietly overwritten.

One thing remains unverified and is flagged as such: Q1/Q2's pin mapping comes
from KiCad's Q_PNP_BEC and the orientation against Figure 10 has not been checked
against the drawing.

470/470 netcheck, 0 unintended, 125 nets.
Parts:
- added C75, C77: 100pF, vuulgaris:C0603, symbol vuulgaris:CC0603JRX7R8BB104
- added C76, C78: 10uF, vuulgaris:C0805, symbol vuulgaris:CC0603JRX7R8BB104
- added Q1, Q2: BC857, vuulgaris:SOT-23, symbol vuulgaris:Q_PNP_BEC
- added R60, R63, R64: 100k, vuulgaris:R0603, symbol vuulgaris:RT0603BRD075K1L
- added R61, R65: 270k, vuulgaris:R0603, symbol vuulgaris:RT0603BRD075K1L
- added R62, R66: 1k, vuulgaris:R0603, symbol vuulgaris:RT0603BRD075K1L
- added R67: 3k, vuulgaris:R0603, symbol vuulgaris:RT0603BRD075K1L
- added R68: 10k, vuulgaris:R0603, symbol vuulgaris:RT0603BRD075K1L
- R40, R41, R42, R44: value 100k -> 20k
- R43: value 100k -> RT0603BRD075K1L
- R45: value 47k -> 20k
- R46: value 56k -> 20k
- R58: value 100k -> 5.6k
Connections:
- net BBD_L_CV: now also C76.2; no longer R43.2
- net BBD_R_CV: now also C78.2; no longer R59.2
- net BBD_R_MIX: no longer R58.2
- net BBD_R_SUM: no longer R58.1
- net DAC_L: now also R59.1; no longer R43.1
- net DAC_R: now also R63.1; no longer R59.1
- net GND: now also R68.2; no longer U12.1 (MODE)
- net NEG12V: now also R58.2, R61.1, R65.1
- net POS12V: now also R67.1
- net U9_C_N renamed BBD_L_EXIN
- net BBD_L_EXIN: now also R59.2, C75.1, R60.1, R61.2; no longer U9.8 (OUT_C)
- net U9_D_N renamed BBD_R_EXIN
- net BBD_R_EXIN: now also C77.1, R63.2, R64.1, R65.2; no longer U9.14 (OUT_D)
- new net BBD_L_CLMP: C76.1, Q1.2 (E), R62.2
- new net BBD_L_EXO: C75.2, Q1.3 (C), R60.2, R62.1, U9.8 (OUT_C)
- new net BBD_R_CLMP: C78.1, Q2.2 (E), R66.2
- new net BBD_R_EXO: C77.2, Q2.3 (C), R64.2, R66.1, U9.14 (OUT_D)
- new net MODE_M: R58.1, U12.1 (MODE)
- new net VCLAMP: Q1.1 (B), Q2.1 (B), R67.2, R68.1
- no-connect marks 132 -> 134

Commit message: hardware: scrap the SSI2100 block, six dual-gang analog pots for filter + delay
Removes 103 parts -- the entire SSI2100 BBD block (U8-U13, Q1/Q2, the filters,
the VCA mix, the MCP4728, the test points and bypass headers) plus ENC9/ENC10.
Netmap goes 160 -> 55 parts, 470 -> 207 connections, verified 207/207 with
nothing unintended. The Daisy's D3/D4 are released, and U4 gains four GPIO back
from the encoders on top of the five it already had spare.

The delay becomes Moritz Klein's mki x es.edu BBD design used as-is: V3205SD,
4096 stages, CD4046 clock, TL072s. Its manual is in docs/.

ENC9/ENC10 were the envelope attack/release pair and they became pots. The
envelope group was already three columns by two rows, so nothing on the panel
moved -- column 0 simply stopped being encoders. Eight encoders now, not ten.

Six ANALOG pots, all DUAL-GANG so one knob moves both stereo sides:

  RV1 CUTOFF          RV2 RESONANCE       RV3 FILTER CV AMT   -> LPG
  RV4 TIME            RV5 FEEDBACK        RV6 WET/DRY         -> BBD

RV2-RV4 were single-gang RK09D and are now RK09L1240A12 like RV1, so all six
share one ORIGIN_OFFSET of (0,-4.83) instead of two values.

place.py currently reports RV4/RV5/RV6 shaft mismatches and 87 orphans over the
board outline. Both are correct: the board still carries the old footprints and
the deleted parts, because only the schematic knows about this yet. F8 resolves
both, and the shaft check is exactly the guard that should complain until it does.
Parts:
- removed C40, C48, C61: 4.7uF, vuulgaris:C0805, symbol vuulgaris:CC0603JRX7R8BB104
- removed C41, C46, C54, C59: 3.3uF, vuulgaris:C0805, symbol vuulgaris:CC0603JRX7R8BB104
- removed C42, C43, C51, C55, C56, C64: 470pF, vuulgaris:C0603, symbol vuulgaris:CC0603JRX7R8BB104
- removed C44, C57: 47pF, vuulgaris:C0603, symbol vuulgaris:CC0603JRX7R8BB104
- removed C45, C58: 1nF, vuulgaris:C0603, symbol vuulgaris:CC0603JRX7R8BB104
- removed C47, C60, C67, C68, C69, C70, C71, C72, C73, C74: 100nF, vuulgaris:C0603, symbol vuulgaris:CC0603JRX7R8BB104
- removed C49, C62: 330pF, vuulgaris:C0603, symbol vuulgaris:CC0603JRX7R8BB104
- removed C50, C63: 390pF, vuulgaris:C0603, symbol vuulgaris:CC0603JRX7R8BB104
- removed C52, C65: 33pF, vuulgaris:C0603, symbol vuulgaris:CC0603JRX7R8BB104
- removed C53, C66, C75, C77: 100pF, vuulgaris:C0603, symbol vuulgaris:CC0603JRX7R8BB104
- removed C76, C78: 10uF, vuulgaris:C0805, symbol vuulgaris:CC0603JRX7R8BB104
- removed ENC10, ENC9: EC12E2430803, vuulgaris:SW-TH_EC12EXXXX, symbol vuulgaris:EC12E2430803
- removed J12, J13: BYPASS, vuulgaris:PinHeader_1x03_P2.54mm_Vertical, symbol vuulgaris:Conn_01x03
- removed Q1, Q2: BC857, vuulgaris:SOT-23, symbol vuulgaris:Q_PNP_BEC
- removed R26: 18.2k, vuulgaris:R0603, symbol vuulgaris:RT0603BRD075K1L
- removed R27: 32.4k, vuulgaris:R0603, symbol vuulgaris:RT0603BRD075K1L
- removed R28, R32, R48, R56, R57, R59, R60, R63, R64: 100k, vuulgaris:R0603, symbol vuulgaris:RT0603BRD075K1L
- removed R29: 47k, vuulgaris:R0603, symbol vuulgaris:RT0603BRD075K1L
- removed R30: 56k, vuulgaris:R0603, symbol vuulgaris:RT0603BRD075K1L
- removed R31, R38, R47, R54: 33k, vuulgaris:R0603, symbol vuulgaris:RT0603BRD075K1L
- removed R33, R49: 100R, vuulgaris:R0603, symbol vuulgaris:RT0603BRD075K1L
- removed R34, R50: 49.9k, vuulgaris:R0603, symbol vuulgaris:RT0603BRD075K1L
- removed R35, R51: 43k, vuulgaris:R0603, symbol vuulgaris:RT0603BRD075K1L
- removed R36, R37, R52, R53: 39k, vuulgaris:R0603, symbol vuulgaris:RT0603BRD075K1L
- removed R39, R55: 120k, vuulgaris:R0603, symbol vuulgaris:RT0603BRD075K1L
- removed R40, R41, R42, R44, R45, R46: 20k, vuulgaris:R0603, symbol vuulgaris:RT0603BRD075K1L
- removed R43: RT0603BRD075K1L, vuulgaris:R0603, symbol vuulgaris:RT0603BRD075K1L
- removed R58: 5.6k, vuulgaris:R0603, symbol vuulgaris:RT0603BRD075K1L
- removed R61, R65: 270k, vuulgaris:R0603, symbol vuulgaris:RT0603BRD075K1L
- removed R62, R66: 1k, vuulgaris:R0603, symbol vuulgaris:RT0603BRD075K1L
- removed R67: 3k, vuulgaris:R0603, symbol vuulgaris:RT0603BRD075K1L
- removed R68: 10k, vuulgaris:R0603, symbol vuulgaris:RT0603BRD075K1L
- removed RV2, RV3, RV4: RK09D117000C, vuulgaris:RES-ADJ-TH_RK09D1130C4G, symbol vuulgaris:RK09D117000C
- removed RV5, RV6: 5k, vuulgaris:Potentiometer_Bourns_3266W_Vertical, symbol vuulgaris:TRIMPOT_3T
- removed TP1, TP10, TP2, TP3, TP4, TP5, TP6, TP7, TP8, TP9: TP, vuulgaris:TestPoint_Pad_D1.5mm, symbol vuulgaris:TestPoint
- removed U10, U11: SSI2100, vuulgaris:SOIC-8_L4.9-W3.9-P1.27-LS6.0-BL, symbol vuulgaris:SSI2100
- removed U12: SSI2164, vuulgaris:SOIC-16_3.9x9.9mm_P1.27mm, symbol vuulgaris:SSI2164
- removed U13: MCP4728, vuulgaris:MSOP-10_3x3mm_P0.5mm, symbol vuulgaris:MCP4728
- removed U8, U9: TL074, vuulgaris:SOIC-14_3.9x8.7mm_P1.27mm, symbol vuulgaris:TL074_FLAT
- added RV2: RESONANCE, vuulgaris:RES-ADJ-TH_RK09L1240A12, symbol vuulgaris:RK09L1240A12
- added RV3: FILTER CV AMT, vuulgaris:RES-ADJ-TH_RK09L1240A12, symbol vuulgaris:RK09L1240A12
- added RV4: TIME, vuulgaris:RES-ADJ-TH_RK09L1240A12, symbol vuulgaris:RK09L1240A12
- added RV5: FEEDBACK, vuulgaris:RES-ADJ-TH_RK09L1240A12, symbol vuulgaris:RK09L1240A12
- added RV6: WET/DRY, vuulgaris:RES-ADJ-TH_RK09L1240A12, symbol vuulgaris:RK09L1240A12
- RV1: value RK09L1240A12 -> CUTOFF
Connections:
- net at SW2.1 (A): now also RV6.1
- net at SW2.2 (B): now also RV6.7
- net at SW2.3 (C): now also RV6.4
- net at SW1.1 (A): now also RV3.1
- net at SW1.2 (B): now also RV3.7
- net at SW1.3 (C): now also RV3.4
- net CLK_A: no longer names the net of U1.D3 (SDMMC_D2)
- net CLK_B: no longer names the net of U1.D4 (SDMMC_D1)
- net ENC10_A: no longer names the net of U4.23 (GPA2)
- net ENC10_B: no longer names the net of U4.24 (GPA3)
- net ENC9_A: no longer names the net of U4.21 (GPA0)
- net ENC9_B: no longer names the net of U4.22 (GPA1)
- no-connect marks 134 -> 150
