File: hardware/kicad/vuulgaris.kicad_sch (KiCad schematic)
At the start: 71 parts, among them J1 TFPUSH, J10 PJ-603_C41409498, J11 TYPE-C-31-M-12, J2 PJ-376, J3 PJ-376, J4 PJ-376, J5 PJ-376, J7 PJ-603_C41409498, J8 PJ-603_C41409498, J9 PJ-603_C41409498, SW1 SW_DPDT_x2, SW2 SW_DPDT_x2, SW4 CPG151101S03, SW5 CPG151101S03, SW6 CPG151101S03, SW7 CPG151101S03, U1 ES_DAISY_PATCH_SM_REV1, U3 MCP23017-E_SO, U4 MCP23017-E_SO, U5 AMS1117-3.3, U6 AMS1117-3.3, U7 DKM10E-12

Commit message: hardware: stereo BBD delay, transcribed from the mki x es.edu schematic
Page 61 of the module manual, two channels, one CD4046 clock each. Not a shared
clock: the dual-gang TIME pot mistracks by a few percent and that mismatch IS
the stereo image, where one clock would give two identical delays that sum to
mono. netmap goes 55 refs / 207 connections -> 164 / 506, verified 506/506
against KiCad's own netlister in both directions, nothing unintended.

The sheet is vector art with no text layer, so it was read from renders rather
than extraction. docs/bbd-mki.md is the readable transcription and the thing to
check the netmap against; it records which junctions were confirmed as hops at
2000dpi and reconciles against the manual's own BOM.

Symbols: CD4046B, TL072, 78L05, MMBFJ113 and 1N4148W from LCSC. The V3205SD is
hand-built, because its "Special 8-Lead Dual-In-Line" package is a DIP-14 lead
pattern with the middle three positions per side omitted -- pads sit at DIP-14
positions 1,2,6,7,8,9,13,14 and are numbered 1-8. A stock DIP-8 would put every
pad in the wrong place; a stock DIP-14 would put them in the right places under
the wrong numbers, which no check downstream would catch.

Two multi-unit symbols had to be flattened. This generator emits one instance
per reference at (unit 1) and cannot express units, so TL072CDR's pins 5/6/7
were never instantiated, and SW_DPDT_x2's two units sit at IDENTICAL symbol
coordinates -- which stubbed the TIME RANGE switch's poles onto each other and
bound U204.6 to BBD_C1A_L, tying the two channels' timing capacitors together.
TL072_FLAT and SW_DPDT_FLAT have all pins at distinct points. SW1/SW2 moved
across too, where the same defect was latent because they are unwired.

Also fixes SW1/SW2 sitting at RV3/RV6's exact sheet coordinates. SW_DPDT_x2 pin
1 is at (5.08, 2.54), which is RK09L1240A12 pin 1, so the LPG SOURCE switch was
shorted onto the dry audio bus in both channels -- invisible until RV6 got nets.

TIME RANGE is not f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
Parts:
- removed SW1, SW2: SW_DPDT_x2, vuulgaris:SW-TH_DW3_DPDT_2MD1T1B1M2QES, symbol vuulgaris:SW_DPDT_x2
- added C105, C106, C107, C108, C109, C111, C121, C122, C205, C206, C207, C208, C209, C211, C221, C222, C40, C41: 100nF, vuulgaris:C0603, symbol vuulgaris:C
- added C110, C210, C42: 3.3uF, vuulgaris:C0805, symbol vuulgaris:C
- added C113, C120, C213, C220: 1uF film, vuulgaris:C0805, symbol vuulgaris:C
- added C114, C214: 1nF C0G, vuulgaris:C0603, symbol vuulgaris:C
- added C116, C216: 220pF C0G, vuulgaris:C0603, symbol vuulgaris:C
- added C119, C219: 15nF C0G 0805, vuulgaris:C0805, symbol vuulgaris:C
- added D103, D104, D105, D106, D107, D203, D204, D205, D206, D207: 1N4148W, vuulgaris:SOD-123_L2.8-W1.8-LS3.7-RD, symbol vuulgaris:1N4148WT4
- added Q1, Q2: J113 / MMBFJ113, vuulgaris:SOT-23-3_L2.9-W1.3-P1.90-LS2.4-BR, symbol vuulgaris:MMBFJ113
- added R104, R204: 0R (IN GAIN -- OPEN, see docs/bbd-mki.md), vuulgaris:R0603, symbol vuulgaris:R
- added R106, R115, R116, R117, R122, R124, R125, R128, R130, R206, R215, R216, R217, R222, R224, R225, R228, R230: 100k, vuulgaris:R0603, symbol vuulgaris:R
- added R107, R207: 1k, vuulgaris:R0603, symbol vuulgaris:R
- added R110, R111, R129, R210, R211, R229: 22k, vuulgaris:R0603, symbol vuulgaris:R
- added R112, R212: 82k, vuulgaris:R0603, symbol vuulgaris:R
- added R113, R213: 47k, vuulgaris:R0603, symbol vuulgaris:R
- added R114, R214: 51k, vuulgaris:R0603, symbol vuulgaris:R
- added R118, R126, R218, R226: 10k, vuulgaris:R0603, symbol vuulgaris:R
- added R119, R219: 4.7k, vuulgaris:R0603, symbol vuulgaris:R
- added R120, R220: 62k, vuulgaris:R0603, symbol vuulgaris:R
- added R121, R221: 2.2M, vuulgaris:R0603, symbol vuulgaris:R
- added R123, R223: 39k, vuulgaris:R0603, symbol vuulgaris:R
- added R127, R227: 6.2k, vuulgaris:R0603, symbol vuulgaris:R
- added R131, R132, R231, R232: 470R, vuulgaris:R0603, symbol vuulgaris:R
- added SW1, SW2: SW_DPDT_FLAT, vuulgaris:SW-TH_DW3_DPDT_2MD1T1B1M2QES, symbol vuulgaris:SW_DPDT_FLAT
- added U101, U201: V3205SD, vuulgaris:DIP-8_SPECIAL_V3205SD, symbol vuulgaris:V3205SD
- added U102, U103, U106, U202, U203, U206: TL072_FLAT, vuulgaris:SOIC-8_L4.9-W3.9-P1.27-LS6.1-BL, symbol vuulgaris:TL072_FLAT
- added U104, U204: CD4046B, vuulgaris:SO-16_L10.3-W5.3-P1.27-LS7.8-BL, symbol vuulgaris:CD4046BNSR
- added U8: 78L05, vuulgaris:SOT-89-3_L4.5-W2.5-P1.50-LS4.2-BR, symbol vuulgaris:78L05_C181132
Connections:
- net GND: now also RV5.1, RV5.4, C105.2, C106.2, C107.2, C108.2, C109.2, C110.2, C111.2, C119.2, C121.2, C122.2, C205.2, C206.2, C207.2, C208.2, C209.2, C210.2, C211.2, C219.2, C221.2, C222.2, C40.2, C41.2, C42.2, D105.2 (A), D106.2 (A), D205.2 (A), D206.2 (A), R106.2, R111.2, R120.2, R121.2, R122.2, R123.2, R124.2, R126.2, R127.2, R129.2, R206.2, R211.2, R220.2, R221.2, R222.2, R223.2, R224.2, R226.2, R227.2, R229.2, U101.1 (GND), U103.3 (1IN+), U104.8 (VSS), U201.1 (GND), U203.3 (1IN+), U204.8 (VSS), U8.2 (GND)
- net NEG12V: now also C106.1, C108.1, C122.1, C206.1, C208.1, C222.1, R113.1, R213.1, U102.4 (V-), U103.4 (V-), U106.4 (V-), U202.4 (V-), U203.4 (V-), U206.4 (V-)
- net POS12V: now also C105.1, C107.1, C121.1, C205.1, C207.1, C221.1, C40.1, R110.1, R125.1, R210.1, R225.1, U102.8 (V+), U103.8 (V+), U106.8 (V+), U202.8 (V+), U203.8 (V+), U206.8 (V+), U8.3 (IN)
- net BBD_DRY_L: now reaches RV6.1
- net BBD_DRY_L: now also R104.1, U102.1 (1OUT), U102.2 (1IN-)
- net BBD_DRY_R: now reaches RV6.4
- net BBD_DRY_R: now also R204.1, U202.1 (1OUT), U202.2 (1IN-)
- net BBD_FB_L: now reaches RV5.2
- net BBD_FB_L: now also R112.1
- net BBD_WETAC_L: now reaches RV5.3
- net BBD_WETAC_L: now also RV6.3, C120.2, R132.1
- net BBD_FB_R: now reaches RV5.5
- net BBD_FB_R: now also R212.1
- net BBD_WETAC_R: now reaches RV5.6
- net BBD_WETAC_R: now also RV6.6, C220.2, R232.1
- net BBD_MIXW_L: now reaches RV6.2
- net BBD_MIXW_L: now also U103.5 (2IN+)
- net BBD_MIXW_R: now reaches RV6.5
- net BBD_MIXW_R: now also U203.5 (2IN+)
- net BBD_TIMEHI_L: now reaches RV4.1
- net BBD_TIMEHI_L: now also R110.2
- net BBD_TIMEW_L: now reaches RV4.2
- net BBD_TIMEW_L: now also R115.1
- net BBD_TIMELO_L: now reaches RV4.3
- net BBD_TIMELO_L: now also R111.1
- net BBD_TIMEHI_R: now reaches RV4.4
- net BBD_TIMEHI_R: now also R210.2
- net BBD_TIMEW_R: now reaches RV4.5
- net BBD_TIMEW_R: now also R215.1
- net BBD_TIMELO_R: now reaches RV4.6
- net BBD_TIMELO_R: now also R211.1
- net CV_OUT_JACK renamed TIME_CV
- net TIME_CV: now also R116.1, R216.1
- new net BBD_AC_L: C113.2, R124.1, U106.3 (1IN+)
- new net BBD_AC_R: C213.2, R224.1, U206.3 (1IN+)
- new net BBD_C1A_L: C114.1, U104.6 (CI(1))
- new net BBD_C1A_R: C214.1, U204.6 (CI(1))
- new net BBD_C1B_L: C114.2, U104.7 (CI(2))
- new net BBD_C1B_R: C214.2, U204.7 (CI(2))
- new net BBD_CLKN_L: U101.2 (CP2), U104.2 (PHASECOMPIOUT)
- new net BBD_CLKN_R: U201.2 (CP2), U204.2 (PHASECOMPIOUT)
- new net BBD_CLK_L: C116.1, U101.6 (CP1), U104.3 (COMPIN), U104.4 (VCOOUT)
- new net BBD_CLK_R: C216.1, U201.6 (CP1), U204.3 (COMPIN), U204.4 (VCOOUT)
- new net BBD_GAIN_L: R104.2, R114.1
- new net BBD_GAIN_R: R204.2, R214.1
- new net BBD_INF_L: R107.2, U102.3 (1IN+)
- new net BBD_INF_R: R207.2, U202.3 (1IN+)
- new net BBD_INHCV_L: R117.1
- new net BBD_INHCV_R: R217.1
- new net BBD_INH_L: D104.2 (A), D106.1 (K), R117.2, U104.5 (INHIBIT)
- new net BBD_INH_R: D204.2 (A), D206.1 (K), R217.2, U204.5 (INHIBIT)
- new net BBD_IN_L: R106.1, R107.1
- new net BBD_IN_R: R206.1, R207.1
- new net BBD_MIX_L: R131.1, U103.6 (2IN-), U103.7 (2OUT)
- new net BBD_MIX_R: R231.1, U203.6 (2IN-), U203.7 (2OUT)
- new net BBD_OUT_L: R131.2
- new net BBD_OUT_R: R231.2
- new net BBD_RAW_L: C113.1, R122.1, U101.4 (OUT2)
- new net BBD_RAW_R: C213.1, R222.1, U201.4 (OUT2)
- new net BBD_SH_FB_L: R129.1, R130.1, U106.6 (2IN-)
- new net BBD_SH_FB_R: R229.1, R230.1, U206.6 (2IN-)
- new net BBD_SH_G_L: D107.2 (A), Q1.3 (G), R128.2
- new net BBD_SH_G_R: D207.2 (A), Q2.3 (G), R228.2
- new net BBD_SH_HOLD_L: C119.1, Q1.2 (S), U106.5 (2IN+)
- new net BBD_SH_HOLD_R: C219.1, Q2.2 (S), U206.5 (2IN+)
- new net BBD_SH_IN_L: Q1.1 (D), R128.1, U106.1 (1OUT), U106.2 (1IN-)
- new net BBD_SH_IN_R: Q2.1 (D), R228.1, U206.1 (1OUT), U206.2 (1IN-)
- new net BBD_SIGIN_L: R118.2, U101.7 (IN), U103.1 (1OUT)
- new net BBD_SIGIN_R: R218.2, U201.7 (IN), U203.1 (1OUT)
- new net BBD_SUM_L: R112.2, R113.2, R114.2, R118.1, U103.2 (1IN-)
- new net BBD_SUM_R: R212.2, R213.2, R214.2, R218.1, U203.2 (1IN-)
- new net BBD_TRIGIN_L: C116.2, R127.1, U102.5 (2IN+)
- new net BBD_TRIGIN_R: C216.2, R227.1, U202.5 (2IN+)
- new net BBD_TRIGREF_L: R125.2, R126.1, U102.6 (2IN-)
- new net BBD_TRIGREF_R: R225.2, R226.1, U202.6 (2IN-)
- new net BBD_TRIG_L: D107.1 (K), U102.7 (2OUT)
- new net BBD_TRIG_R: D207.1 (K), U202.7 (2OUT)
- new net BBD_VCOCV_L: D103.2 (A), D105.1 (K), R115.2, R116.2, U104.9 (VCOIN)
- new net BBD_VCOCV_R: D203.2 (A), D205.1 (K), R215.2, R216.2, U204.9 (VCOIN)
- new net BBD_VCOR1_L: R123.1, U104.11 (R1TOVSS)
- new net BBD_VCOR1_R: R223.1, U204.11 (R1TOVSS)
- new net BBD_VCOR2_L: R121.1, U104.12 (R2TOVSS)
- new net BBD_VCOR2_R: R221.1, U204.12 (R2TOVSS)
- new net BBD_VGG_L: C110.1, R119.2, R120.1, U101.8 (VGG)
- new net BBD_VGG_R: C210.1, R219.2, R220.1, U201.8 (VGG)
- new net BBD_WETOUT_L: R132.2
- new net BBD_WETOUT_R: R232.2
- new net BBD_WET_L: C120.1, R130.2, U106.7 (2OUT)
- new net BBD_WET_R: C220.1, R230.2, U206.7 (2OUT)
- new net P5V_BBD: C109.1, C111.1, C209.1, C211.1, C41.1, C42.1, D103.1 (K), D104.1 (K), D203.1 (K), D204.1 (K), R119.1, R219.1, U101.5 (VDD), U104.14 (SIGNALIN), U104.16 (VDD), U201.5 (VDD), U204.14 (SIGNALIN), U204.16 (VDD), U8.1 (OUT)
- no-connect marks 150 -> 142
