File: hardware/kicad/vuulgaris.kicad_sch (KiCad schematic)
At the start: 291 parts, among them J1 TFPUSH, J10 PJ-603_C41409498, J11 TYPE-C-31-M-12, J12 FACEPLATE 2x5 IDC, J2 PJ-376, J3 PJ-376, J4 PJ-376, J5 PJ-376, J6 PJ-376, J7 PJ-603_C41409498, J8 PJ-603_C41409498, J9 PJ-603_C41409498, Q1 J113 / MMBFJ113, Q2 J113 / MMBFJ113, SW1 SW_DPDT_FLAT, SW2 SW_DPDT_FLAT, SW4 12x12 tactile, SW5 12x12 tactile, SW6 12x12 tactile, SW7 12x12 tactile, SW8 12x12 tactile, SW9 12x12 tactile, U1 ES_DAISY_PATCH_SM_REV1, U101 V3205SD, U102 TL072_FLAT, U103 TL072_FLAT, U104 CD4046B, U106 TL072_FLAT, U201 V3205SD, U202 TL072_FLAT, U203 TL072_FLAT, U204 CD4046B, U206 TL072_FLAT, U3 MCP23017-E_SO, U301 TL084, U302 TL074, U4 MCP23017-E_SO, U401 TL084, U402 TL074, U5 AMS1117-3.3, U6 AMS1117-3.3, U7 DKM10E-12, U8 78L05, U9 OPA1688_FLAT

Commit message: hardware: drop the 1/4" outs to line level, fix the headphone series R
The 1/4" outs sat straight on BBD_OUT at Eurorack level, 9.5Vpp / +12.7dBu.
That survives a pro interface but clips consumer gear and anything with an
instrument input. R513-R516 divide it to +3.9dBu full scale.

The divider sits downstream of the C503 (resample) and C505 (headphone) taps,
so BBD_OUT keeps the Eurorack level the internal chain is matched to and only
the jack moves. With R131's existing 470R the ratio is 1000/2770 = -8.85dB,
639R out, 2770R load on U103 -- inside the TL072's 2k rating.

R511/R512 22R -> 4R7. They are outside U9's feedback loop, so they set output
impedance directly: 22R into 32R cans is damping factor 1.5, which colours the
bass differently for every pair, and throws away 4.6dB. The OPA1688 is a
headphone driver with internal short-circuit protection and does not need the
isolation.

pose.py is new. place.py owns X/Y but not layer or rotation, so every F8 drops
re-imported footprints back on F.Cu at 0 degrees -- that has eaten the bypass
caps once and the headphone block twice. pose.py snapshots and restores all
295 poses; verified by clobbering the 160 non-default ones and restoring
byte-identical. It derives pad angles from the board rather than the library,
because a library lookup miss invents a rotation out of nothing.

Documented that back-side silkscreen text is unmirrored on ~160 parts: 324
fp_text entries disagree with their own layer, so back reference designators
will plot reversed. Cosmetic, not fixed here.
Parts:
- added R513, R515: 1k3, vuulgaris:R0603, symbol vuulgaris:R
- added R514, R516: 1k, vuulgaris:R0603, symbol vuulgaris:R
- R511, R512: value 22R -> 4R7
Connections:
- net BBD_OUT_L: now also R513.1; no longer J9.4
- net BBD_OUT_R: now also R515.1; no longer J10.4
- net GND: now also R514.2, R516.2
- new net LINE_OUT_L: J9.4, R513.2, R514.1
- new net LINE_OUT_R: J10.4, R515.2, R516.1
Changed lines of the file:
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@@
     (in_bom yes) (on_board yes) (dnp no)
     (property "Reference" "R511" (at 1160 3828 0) (effects (font (size 1.27 1.27))))
-    (property "Value" "22R" (at 1160 3831 0) (effects (font (size 1.27 1.27))))
+    (property "Value" "4R7" (at 1160 3831 0) (effects (font (size 1.27 1.27))))
     (property "Footprint" "vuulgaris:R0603" (at 1160 3840 0) (effects (font (size 1.27 1.27)) hide))
     (property "Datasheet" "" (at 1160 3840 0) (effects (font (size 1.27 1.27)) hide))
@@
     (in_bom yes) (on_board yes) (dnp no)
     (property "Reference" "R512" (at 1290 3828 0) (effects (font (size 1.27 1.27))))
-    (property "Value" "22R" (at 1290 3831 0) (effects (font (size 1.27 1.27))))
+    (property "Value" "4R7" (at 1290 3831 0) (effects (font (size 1.27 1.27))))
     (property "Footprint" "vuulgaris:R0603" (at 1290 3840 0) (effects (font (size 1.27 1.27)) hide))
     (property "Datasheet" "" (at 1290 3840 0) (effects (font (size 1.27 1.27)) hide))
@@
     (pin "2")
   )
+  (symbol (lib_id "vuulgaris:R") (at 120 3930 0) (unit 1)
+    (in_bom yes) (on_board yes) (dnp no)
+    (property "Reference" "R513" (at 120 3918 0) (effects (font (size 1.27 1.27))))
+    (property "Value" "1k3" (at 120 3921 0) (effects (font (size 1.27 1.27))))
+    (property "Footprint" "vuulgaris:R0603" (at 120 3930 0) (effects (font (size 1.27 1.27)) hide))
+    (property "Datasheet" "" (at 120 3930 0) (effects (font (size 1.27 1.27)) hide))
+    (pin "1")
+    (pin "2")
+  )
+  (symbol (lib_id "vuulgaris:R") (at 250 3930 0) (unit 1)
+    (in_bom yes) (on_board yes) (dnp no)
+    (property "Reference" "R514" (at 250 3918 0) (effects (font (size 1.27 1.27))))
+    (property "Value" "1k" (at 250 3921 0) (effects (font (size 1.27 1.27))))
+    (property "Footprint" "vuulgaris:R0603" (at 250 3930 0) (effects (font (size 1.27 1.27)) hide))
+    (property "Datasheet" "" (at 250 3930 0) (effects (font (size 1.27 1.27)) hide))
+    (pin "1")
+    (pin "2")
+  )
+  (symbol (lib_id "vuulgaris:R") (at 380 3930 0) (unit 1)
+    (in_bom yes) (on_board yes) (dnp no)
+    (property "Reference" "R515" (at 380 3918 0) (effects (font (size 1.27 1.27))))
+    (property "Value" "1k3" (at 380 3921 0) (effects (font (size 1.27 1.27))))
+    (property "Footprint" "vuulgaris:R0603" (at 380 3930 0) (effects (font (size 1.27 1.27)) hide))
+    (property "Datasheet" "" (at 380 3930 0) (effects (font (size 1.27 1.27)) hide))
+    (pin "1")
+    (pin "2")
+  )
+  (symbol (lib_id "vuulgaris:R") (at 510 3930 0) (unit 1)
+    (in_bom yes) (on_board yes) (dnp no)
+    (property "Reference" "R516" (at 510 3918 0) (effects (font (size 1.27 1.27))))
+    (property "Value" "1k" (at 510 3921 0) (effects (font (size 1.27 1.27))))
+    (property "Footprint" "vuulgaris:R0603" (at 510 3930 0) (effects (font (size 1.27 1.27)) hide))
+    (property "Datasheet" "" (at 510 3930 0) (effects (font (size 1.27 1.27)) hide))
+    (pin "1")
+    (pin "2")
+  )
   (symbol (lib_id "vuulgaris:TRIMPOT_3T") (at 520 3900 0) (unit 1)
     (in_bom yes) (on_board yes) (dnp no)
@@
   (wire (pts (xy 1290.0 3836.19) (xy 1290.0 3826.03)) (stroke (width 0) (type solid)))
   (wire (pts (xy 1290.0 3843.81) (xy 1290.0 3853.97)) (stroke (width 0) (type solid)))
+  (wire (pts (xy 120.0 3926.19) (xy 120.0 3916.03)) (stroke (width 0) (type solid)))
+  (wire (pts (xy 120.0 3933.81) (xy 120.0 3943.97)) (stroke (width 0) (type solid)))
+  (wire (pts (xy 250.0 3926.19) (xy 250.0 3916.03)) (stroke (width 0) (type solid)))
+  (wire (pts (xy 250.0 3933.81) (xy 250.0 3943.97)) (stroke (width 0) (type solid)))
+  (wire (pts (xy 380.0 3926.19) (xy 380.0 3916.03)) (stroke (width 0) (type solid)))
+  (wire (pts (xy 380.0 3933.81) (xy 380.0 3943.97)) (stroke (width 0) (type solid)))
+  (wire (pts (xy 510.0 3926.19) (xy 510.0 3916.03)) (stroke (width 0) (type solid)))
+  (wire (pts (xy 510.0 3933.81) (xy 510.0 3943.97)) (stroke (width 0) (type solid)))
   (wire (pts (xy 514.92 3897.46) (xy 504.76 3897.46)) (stroke (width 0) (type solid)))
   (wire (pts (xy 525.08 3900.0) (xy 535.24 3900.0)) (stroke (width 0) (type solid)))
@@
     (effects (font (size 1.27 1.27)) (justify left bottom))
   )
-  (label "BBD_OUT_R" (at 481.51 635.08 0) (fields_autoplaced)
+  (label "LINE_OUT_R" (at 481.51 635.08 0) (fields_autoplaced)
     (effects (font (size 1.27 1.27)) (justify left bottom))
   )
@@
     (effects (font (size 1.27 1.27)) (justify left bottom))
   )
-  (label "BBD_OUT_L" (at 386.51 635.08 0) (fields_autoplaced)
+  (label "LINE_OUT_L" (at 386.51 635.08 0) (fields_autoplaced)
     (effects (font (size 1.27 1.27)) (justify left bottom))
   )
@@
     (effects (font (size 1.27 1.27)) (justify left bottom))
   )
+  (label "BBD_OUT_L" (at 120.0 3916.03 90) (fields_autoplaced)
+    (effects (font (size 1.27 1.27)) (justify left bottom))
+  )
+  (label "LINE_OUT_L" (at 120.0 3943.97 270) (fields_autoplaced)
+    (effects (font (size 1.27 1.27)) (justify left bottom))
+  )
+  (label "LINE_OUT_L" (at 250.0 3916.03 90) (fields_autoplaced)
+    (effects (font (size 1.27 1.27)) (justify left bottom))
+  )
+  (label "GND" (at 250.0 3943.97 270) (fields_autoplaced)
+    (effects (font (size 1.27 1.27)) (justify left bottom))
+  )
+  (label "BBD_OUT_R" (at 380.0 3916.03 90) (fields_autoplaced)
+    (effects (font (size 1.27 1.27)) (justify left bottom))
+  )
+  (label "LINE_OUT_R" (at 380.0 3943.97 270) (fields_autoplaced)
+    (effects (font (size 1.27 1.27)) (justify left bottom))
+  )
+  (label "LINE_OUT_R" (at 510.0 3916.03 90) (fields_autoplaced)
+    (effects (font (size 1.27 1.27)) (justify left bottom))
+  )
+  (label "GND" (at 510.0 3943.97 270) (fields_autoplaced)
+    (effects (font (size 1.27 1.27)) (justify left bottom))
+  )

Commit message: hardware: EXT input preamp, and U9's bypass caps were 15mm away
The 1/4" inputs fed U1.B3/B4 through a coupling cap and nothing else, at unity.
The Patch SM's full scale is Eurorack 9.5Vpp, so a receiver lands at -20dBFS and
a phone at -10dBFS. Software gain does not recover that -- it lifts the
converter's noise floor with the signal.

U10 is a second OPA1688, non-inverting, with RT503/RT504 in the feedback leg
giving 1x to 10.1x. It sits before SW2 so only the EXT branch is gained; the
resample path keeps its Eurorack level. C501 already blocks DC into the switch,
so the feedback leg needs no cap and U10's offset never reaches the module. At
minimum trim the stage is a unity follower, so a hot source is still safe.

R517/R518 1k are series protection off the jacks. There was none at all -- C501
went straight onto a module pin, and a source peaking at +18dBu is 17.4Vpp
against a +/-4.75V input. Against R519's 100k the 1k costs under 0.1dB.

Adding U9 and U10 to place.py's BYPASS table caught C507/C508 sitting 15.5mm and
15.0mm from the pins they decouple -- they were never in the table, so the check
had been auditing only the parts that were already right. RT502 moves 7.5mm off
U9 pin 8 to free the pocket; both caps are now inside 2.5mm.

The slot finder used for all of this had the back-side mirror wrong: place.py
negates local Y for B.Cu footprints and the finder did not, so every proposed
position was judged against mirrored neighbours. It also required quoted pad
names, which the library files do not use, so candidates came back with no
geometry at all and passed. Both fixed, and the placements redone -- R513-R516
moved as a result.
Parts:
- added C509, C510: 100nF, vuulgaris:C0603, symbol vuulgaris:C
- added C511, C512: 1uF film, vuulgaris:C0603, symbol vuulgaris:C
- added R517, R518: 1k, vuulgaris:R0603, symbol vuulgaris:R
- added R519, R520: 100k, vuulgaris:R0603, symbol vuulgaris:R
- added R521, R522: 2k2, vuulgaris:R0603, symbol vuulgaris:R
- added RT503, RT504: 20k trim, vuulgaris:RES-ADJ-SMD_3224W, symbol vuulgaris:TRIMPOT_3T
- added U10: OPA1688_FLAT, vuulgaris:SOP-8_L4.9-W3.9-P1.27-LS6.0-BL, symbol vuulgaris:OPA1688_FLAT
Connections:
- net EXT_IN_L: now also R517.1; no longer C501.1
- net EXT_IN_R: now also R518.1; no longer C502.1
- net GND: now also C509.2, C510.2, R519.2, R520.2, R521.2, R522.2
- net NEG12V: now also C510.1, U10.4 (V-)
- net POS12V: now also C509.1, U10.8 (V+)
- new net EXT_AMP_IN_L: C511.2, R519.1, U10.3 (1IN+)
- new net EXT_AMP_IN_R: C512.2, R520.1, U10.5 (2IN+)
- new net EXT_AMP_OUT_L: C501.1, RT503.1, U10.1 (1OUT)
- new net EXT_AMP_OUT_R: C502.1, RT504.1, U10.7 (2OUT)
- new net EXT_FB_L: R521.1, RT503.2 (WIPER), RT503.3, U10.2 (1IN-)
- new net EXT_FB_R: R522.1, RT504.2 (WIPER), RT504.3, U10.6 (2IN-)
- new net EXT_PROT_L: C511.1, R517.2
- new net EXT_PROT_R: C512.1, R518.2

Commit message: hardware: the 1uF "film" caps are 0805 X7R, because film was never possible
Fourteen caps carried the value "1uF film" in an 0603 footprint, which is not a
shippable part. SMD film tops out near 0.1uF in 1210; 1uF film is a leaded box
cap about 7x7mm on a 5mm pitch, hand-soldered, on a board whose hand-solder list
was cut to four genuinely unsourceable parts. What would actually have been
assembled is a Class II MLCC, so the value string was describing a wish.

They are now 1uF X7R 50V in C0805. Renaming alone would have been honest but
would have left the distortion: Class II voltage-coefficient nonlinearity scales
with the field across the dielectric, and a 1uF 50V part in 0805 has more and
thicker layers than a 1uF 16V part in 0603 being asked to swing a third of its
rating on a +/-4.75V Eurorack signal. 1uF C0G is the linear answer and is not an
option -- nothing below 2220, a few dollars each, fourteen of them would swallow
the board.

Eleven took the bigger footprint where they stood, checked against the corrected
back-side geometry. C505 turns 90 degrees to clear J6's body, C511 moves 3.4mm,
C512 0.25mm.

939/939 connections verified, all 28 bypass caps inside 5.0mm, no pad overlaps,
same-face body overlaps back to the pre-existing four.
Parts:
- C113, C120, C213, C220: value 1uF film -> 1uF X7R 50V
- C306, C406, C501, C502, C503, C504, C505, C506, C511, C512: value 1uF film -> 1uF X7R 50V; footprint vuulgaris:C0603 -> vuulgaris:C0805
Changed lines of the file:
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@@
     (in_bom yes) (on_board yes) (dnp no)
     (property "Reference" "C113" (at 1170 988 0) (effects (font (size 1.27 1.27))))
-    (property "Value" "1uF film" (at 1170 991 0) (effects (font (size 1.27 1.27))))
+    (property "Value" "1uF X7R 50V" (at 1170 991 0) (effects (font (size 1.27 1.27))))
     (property "Footprint" "vuulgaris:C0805" (at 1170 1000 0) (effects (font (size 1.27 1.27)) hide))
     (property "Datasheet" "" (at 1170 1000 0) (effects (font (size 1.27 1.27)) hide))
@@
     (in_bom yes) (on_board yes) (dnp no)
     (property "Reference" "C120" (at 570 1068 0) (effects (font (size 1.27 1.27))))
-    (property "Value" "1uF film" (at 570 1071 0) (effects (font (size 1.27 1.27))))
+    (property "Value" "1uF X7R 50V" (at 570 1071 0) (effects (font (size 1.27 1.27))))
     (property "Footprint" "vuulgaris:C0805" (at 570 1080 0) (effects (font (size 1.27 1.27)) hide))
     (property "Datasheet" "" (at 570 1080 0) (effects (font (size 1.27 1.27)) hide))
@@
     (in_bom yes) (on_board yes) (dnp no)
     (property "Reference" "C213" (at 1170 1688 0) (effects (font (size 1.27 1.27))))
-    (property "Value" "1uF film" (at 1170 1691 0) (effects (font (size 1.27 1.27))))
+    (property "Value" "1uF X7R 50V" (at 1170 1691 0) (effects (font (size 1.27 1.27))))
     (property "Footprint" "vuulgaris:C0805" (at 1170 1700 0) (effects (font (size 1.27 1.27)) hide))
     (property "Datasheet" "" (at 1170 1700 0) (effects (font (size 1.27 1.27)) hide))
@@
     (in_bom yes) (on_board yes) (dnp no)
     (property "Reference" "C220" (at 570 1768 0) (effects (font (size 1.27 1.27))))
-    (property "Value" "1uF film" (at 570 1771 0) (effects (font (size 1.27 1.27))))
+    (property "Value" "1uF X7R 50V" (at 570 1771 0) (effects (font (size 1.27 1.27))))
     (property "Footprint" "vuulgaris:C0805" (at 570 1780 0) (effects (font (size 1.27 1.27)) hide))
     (property "Datasheet" "" (at 570 1780 0) (effects (font (size 1.27 1.27)) hide))
@@
     (in_bom yes) (on_board yes) (dnp no)
     (property "Reference" "C306" (at 770 2988 0) (effects (font (size 1.27 1.27))))
-    (property "Value" "1uF film" (at 770 2991 0) (effects (font (size 1.27 1.27))))
-    (property "Footprint" "vuulgaris:C0603" (at 770 3000 0) (effects (font (size 1.27 1.27)) hide))
+    (property "Value" "1uF X7R 50V" (at 770 2991 0) (effects (font (size 1.27 1.27))))
+    (property "Footprint" "vuulgaris:C0805" (at 770 3000 0) (effects (font (size 1.27 1.27)) hide))
     (property "Datasheet" "" (at 770 3000 0) (effects (font (size 1.27 1.27)) hide))
     (pin "1")
@@
     (in_bom yes) (on_board yes) (dnp no)
     (property "Reference" "C406" (at 770 3288 0) (effects (font (size 1.27 1.27))))
-    (property "Value" "1uF film" (at 770 3291 0) (effects (font (size 1.27 1.27))))
-    (property "Footprint" "vuulgaris:C0603" (at 770 3300 0) (effects (font (size 1.27 1.27)) hide))
+    (property "Value" "1uF X7R 50V" (at 770 3291 0) (effects (font (size 1.27 1.27))))
+    (property "Footprint" "vuulgaris:C0805" (at 770 3300 0) (effects (font (size 1.27 1.27)) hide))
     (property "Datasheet" "" (at 770 3300 0) (effects (font (size 1.27 1.27)) hide))
     (pin "1")
@@
     (in_bom yes) (on_board yes) (dnp no)
     (property "Reference" "C501" (at 120 3738 0) (effects (font (size 1.27 1.27))))
-    (property "Value" "1uF film" (at 120 3741 0) (effects (font (size 1.27 1.27))))
-    (property "Footprint" "vuulgaris:C0603" (at 120 3750 0) (effects (font (size 1.27 1.27)) hide))
+    (property "Value" "1uF X7R 50V" (at 120 3741 0) (effects (font (size 1.27 1.27))))
+    (property "Footprint" "vuulgaris:C0805" (at 120 3750 0) (effects (font (size 1.27 1.27)) hide))
     (property "Datasheet" "" (at 120 3750 0) (effects (font (size 1.27 1.27)) hide))
     (pin "1")
@@
     (in_bom yes) (on_board yes) (dnp no)
     (property "Reference" "C502" (at 250 3738 0) (effects (font (size 1.27 1.27))))
-    (property "Value" "1uF film" (at 250 3741 0) (effects (font (size 1.27 1.27))))
-    (property "Footprint" "vuulgaris:C0603" (at 250 3750 0) (effects (font (size 1.27 1.27)) hide))
+    (property "Value" "1uF X7R 50V" (at 250 3741 0) (effects (font (size 1.27 1.27))))
+    (property "Footprint" "vuulgaris:C0805" (at 250 3750 0) (effects (font (size 1.27 1.27)) hide))
     (property "Datasheet" "" (at 250 3750 0) (effects (font (size 1.27 1.27)) hide))
     (pin "1")
@@
     (in_bom yes) (on_board yes) (dnp no)
     (property "Reference" "C503" (at 380 3738 0) (effects (font (size 1.27 1.27))))
-    (property "Value" "1uF film" (at 380 3741 0) (effects (font (size 1.27 1.27))))
-    (property "Footprint" "vuulgaris:C0603" (at 380 3750 0) (effects (font (size 1.27 1.27)) hide))
+    (property "Value" "1uF X7R 50V" (at 380 3741 0) (effects (font (size 1.27 1.27))))
+    (property "Footprint" "vuulgaris:C0805" (at 380 3750 0) (effects (font (size 1.27 1.27)) hide))
     (property "Datasheet" "" (at 380 3750 0) (effects (font (size 1.27 1.27)) hide))
     (pin "1")
@@
     (in_bom yes) (on_board yes) (dnp no)
     (property "Reference" "C504" (at 510 3738 0) (effects (font (size 1.27 1.27))))
-    (property "Value" "1uF film" (at 510 3741 0) (effects (font (size 1.27 1.27))))
-    (property "Footprint" "vuulgaris:C0603" (at 510 3750 0) (effects (font (size 1.27 1.27)) hide))
+    (property "Value" "1uF X7R 50V" (at 510 3741 0) (effects (font (size 1.27 1.27))))
+    (property "Footprint" "vuulgaris:C0805" (at 510 3750 0) (effects (font (size 1.27 1.27)) hide))
     (property "Datasheet" "" (at 510 3750 0) (effects (font (size 1.27 1.27)) hide))
     (pin "1")
@@
     (in_bom yes) (on_board yes) (dnp no)
     (property "Reference" "C505" (at 640 3738 0) (effects (font (size 1.27 1.27))))
-    (property "Value" "1uF film" (at 640 3741 0) (effects (font (size 1.27 1.27))))
-    (property "Footprint" "vuulgaris:C0603" (at 640 3750 0) (effects (font (size 1.27 1.27)) hide))
+    (property "Value" "1uF X7R 50V" (at 640 3741 0) (effects (font (size 1.27 1.27))))
+    (property "Footprint" "vuulgaris:C0805" (at 640 3750 0) (effects (font (size 1.27 1.27)) hide))
     (property "Datasheet" "" (at 640 3750 0) (effects (font (size 1.27 1.27)) hide))
     (pin "1")
@@
     (in_bom yes) (on_board yes) (dnp no)
     (property "Reference" "C506" (at 770 3738 0) (effects (font (size 1.27 1.27))))
-    (property "Value" "1uF film" (at 770 3741 0) (effects (font (size 1.27 1.27))))
-    (property "Footprint" "vuulgaris:C0603" (at 770 3750 0) (effects (font (size 1.27 1.27)) hide))
+    (property "Value" "1uF X7R 50V" (at 770 3741 0) (effects (font (size 1.27 1.27))))
+    (property "Footprint" "vuulgaris:C0805" (at 770 3750 0) (effects (font (size 1.27 1.27)) hide))
     (property "Datasheet" "" (at 770 3750 0) (effects (font (size 1.27 1.27)) hide))
     (pin "1")
@@
     (in_bom yes) (on_board yes) (dnp no)
     (property "Reference" "C511" (at 120 3828 0) (effects (font (size 1.27 1.27))))
-    (property "Value" "1uF film" (at 120 3831 0) (effects (font (size 1.27 1.27))))
-    (property "Footprint" "vuulgaris:C0603" (at 120 3840 0) (effects (font (size 1.27 1.27)) hide))
+    (property "Value" "1uF X7R 50V" (at 120 3831 0) (effects (font (size 1.27 1.27))))
+    (property "Footprint" "vuulgaris:C0805" (at 120 3840 0) (effects (font (size 1.27 1.27)) hide))
     (property "Datasheet" "" (at 120 3840 0) (effects (font (size 1.27 1.27)) hide))
     (pin "1")
@@
     (in_bom yes) (on_board yes) (dnp no)
     (property "Reference" "C512" (at 250 3828 0) (effects (font (size 1.27 1.27))))
-    (property "Value" "1uF film" (at 250 3831 0) (effects (font (size 1.27 1.27))))
-    (property "Footprint" "vuulgaris:C0603" (at 250 3840 0) (effects (font (size 1.27 1.27)) hide))
+    (property "Value" "1uF X7R 50V" (at 250 3831 0) (effects (font (size 1.27 1.27))))
+    (property "Footprint" "vuulgaris:C0805" (at 250 3840 0) (effects (font (size 1.27 1.27)) hide))
     (property "Datasheet" "" (at 250 3840 0) (effects (font (size 1.27 1.27)) hide))
     (pin "1")
