File: hardware/faceplate/vuulgaris-faceplate.kicad_pcb (KiCad board)
At the start: 4 copper layers, 298.3 x 137.8 mm, 54 parts, among them J1 HX JN2.54-2x5P TP H8.9, U1 MSP430FR2675TPT, Y1 32.768kHz FC-135 12.5pF

Commit message: faceplate: drop the OLED reference drawing from F.Fab
Dylan has seen the window against the pixels and glass; the outlines and
labels are off the board, and mkholes.py no longer draws them (or clears
F.Fab). panelgeo.oled_outlines() went with them. The window cut is
unchanged.

Checked: boardcheck parity 0, clearance 0; DRC --unrouted 0 errors;
panelcheck --strict 13 OK.
Other:
- board text removed: "OLED glass 62.10 x 39.85 -- black past the pixels"
- board text removed: "OLED pixels (active area) 55.01 x 27.49"
Changed lines of the file:
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@@
     )
   )
+  (gr_circle (center 219.143 73.225) (end 222.893 73.225)
+    (stroke (width 0.1) (type default)) (fill none) (layer "Edge.Cuts"))
+  (gr_line (start 368.592857 66.1485) (end 368.592857 98.048499)
+    (stroke (width 0.1) (type default)) (layer "Edge.Cuts"))
+  (gr_circle (center 241.143 89.681) (end 244.893 89.681)
+    (stroke (width 0.1) (type default)) (fill none) (layer "Edge.Cuts"))
+  (gr_circle (center 125.821 143.953) (end 129.420999 143.953)
+    (stroke (width 0.1) (type default)) (fill none) (layer "Edge.Cuts"))
+  (gr_circle (center 280.643 89.631) (end 283.443 89.631)
+    (stroke (width 0.1) (type default)) (fill none) (layer "Edge.Cuts"))
+  (gr_circle (center 169.143 89.851) (end 173.893 89.851)
+    (stroke (width 0.1) (type default)) (fill none) (layer "Edge.Cuts"))
+  (gr_circle (center 191.143 89.851) (end 195.893 89.851)
+    (stroke (width 0.1) (type default)) (fill none) (layer "Edge.Cuts"))
+  (gr_circle (center 141.321 143.953) (end 144.921 143.953)
+    (stroke (width 0.1) (type default)) (fill none) (layer "Edge.Cuts"))
+  (gr_circle (center 293.643 89.631) (end 296.443 89.631)
+    (stroke (width 0.1) (type default)) (fill none) (layer "Edge.Cuts"))
+  (gr_circle (center 141.321 169.353) (end 144.921 169.353)
+    (stroke (width 0.1) (type default)) (fill none) (layer "Edge.Cuts"))
+  (gr_arc (start 367.592857 65.1485) (mid 368.299963 65.441393) (end 368.592857 66.1485)
+    (stroke (width 0.1) (type default)) (layer "Edge.Cuts"))
   (gr_circle (center 169.143 73.395) (end 173.893 73.395)
+    (stroke (width 0.1) (type default)) (fill none) (layer "Edge.Cuts"))
+  (gr_circle (center 191.143 73.395) (end 195.893 73.395)
     (stroke (width 0.1) (type default)) (fill none) (layer "Edge.Cuts"))
   (gr_circle (center 125.821 169.353) (end 129.420999 169.353)
     (stroke (width 0.1) (type default)) (fill none) (layer "Edge.Cuts"))
-  (gr_circle (center 241.143 89.681) (end 244.893 89.681)
-    (stroke (width 0.1) (type default)) (fill none) (layer "Edge.Cuts"))
-  (gr_circle (center 219.143 89.681) (end 222.893 89.681)
-    (stroke (width 0.1) (type default)) (fill none) (layer "Edge.Cuts"))
-  (gr_circle (center 293.643 89.631) (end 296.443 89.631)
-    (stroke (width 0.1) (type default)) (fill none) (layer "Edge.Cuts"))
-  (gr_line (start 308.502515 98.048499) (end 308.502515 66.1485)
-    (stroke (width 0.1) (type default)) (layer "Edge.Cuts"))
-  (gr_circle (center 191.143 73.395) (end 195.893 73.395)
-    (stroke (width 0.1) (type default)) (fill none) (layer "Edge.Cuts"))
-  (gr_circle (center 280.643 89.631) (end 283.443 89.631)
-    (stroke (width 0.1) (type default)) (fill none) (layer "Edge.Cuts"))
-  (gr_circle (center 133.571 125.453) (end 138.571 125.453)
+  (gr_rect (start 100 50) (end 398.285714 187.81)
     (stroke (width 0.1) (type default)) (fill none) (layer "Edge.Cuts"))
   (gr_circle (center 125.143 73.395) (end 129.893 73.395)
+    (stroke (width 0.1) (type default)) (fill none) (layer "Edge.Cuts"))
+  (gr_circle (center 241.143 73.225) (end 244.893 73.225)
     (stroke (width 0.1) (type default)) (fill none) (layer "Edge.Cuts"))
   (gr_circle (center 263.143 89.681) (end 266.893 89.681)
@@
   (gr_line (start 309.502515 65.1485) (end 367.592857 65.1485)
     (stroke (width 0.1) (type default)) (layer "Edge.Cuts"))
-  (gr_circle (center 141.321 169.353) (end 144.921 169.353)
-    (stroke (width 0.1) (type default)) (fill none) (layer "Edge.Cuts"))
   (gr_circle (center 147.143 73.395) (end 151.893 73.395)
     (stroke (width 0.1) (type default)) (fill none) (layer "Edge.Cuts"))
-  (gr_rect (start 100 50) (end 398.285714 187.81)
+  (gr_arc (start 309.502515 99.048499) (mid 308.795409 98.755606) (end 308.502515 98.048499)
+    (stroke (width 0.1) (type default)) (layer "Edge.Cuts"))
+  (gr_arc (start 368.592857 98.048499) (mid 368.299963 98.755606) (end 367.592857 99.048499)
+    (stroke (width 0.1) (type default)) (layer "Edge.Cuts"))
+  (gr_circle (center 125.143 89.851) (end 129.893 89.851)
     (stroke (width 0.1) (type default)) (fill none) (layer "Edge.Cuts"))
   (gr_circle (center 125.821 156.653) (end 129.420999 156.653)
     (stroke (width 0.1) (type default)) (fill none) (layer "Edge.Cuts"))
-  (gr_circle (center 241.143 73.225) (end 244.893 73.225)
+  (gr_circle (center 141.321 156.653) (end 144.921 156.653)
     (stroke (width 0.1) (type default)) (fill none) (layer "Edge.Cuts"))
-  (gr_arc (start 309.502515 99.048499) (mid 308.795409 98.755606) (end 308.502515 98.048499)
+  (gr_line (start 308.502515 98.048499) (end 308.502515 66.1485)
+    (stroke (width 0.1) (type default)) (layer "Edge.Cuts"))
+  (gr_circle (center 219.143 89.681) (end 222.893 89.681)
+    (stroke (width 0.1) (type default)) (fill none) (layer "Edge.Cuts"))
+  (gr_circle (center 147.143 89.851) (end 151.893 89.851)
+    (stroke (width 0.1) (type default)) (fill none) (layer "Edge.Cuts"))
+  (gr_arc (start 308.502515 66.1485) (mid 308.795409 65.441393) (end 309.502515 65.1485)
+    (stroke (width 0.1) (type default)) (layer "Edge.Cuts"))
+  (gr_circle (center 133.571 125.453) (end 138.571 125.453)
+    (stroke (width 0.1) (type default)) (fill none) (layer "Edge.Cuts"))
+  (gr_line (start 367.592857 99.048499) (end 309.502515 99.048499)
     (stroke (width 0.1) (type default)) (layer "Edge.Cuts"))
   (gr_circle (center 263.143 73.225) (end 266.893 73.225)
     (stroke (width 0.1) (type default)) (fill none) (layer "Edge.Cuts"))
-  (gr_arc (start 308.502515 66.1485) (mid 308.795409 65.441393) (end 309.502515 65.1485)
-    (stroke (width 0.1) (type default)) (layer "Edge.Cuts"))
-  (gr_circle (center 125.143 89.851) (end 129.893 89.851)
-    (stroke (width 0.1) (type default)) (fill none) (layer "Edge.Cuts"))
-  (gr_line (start 367.592857 99.048499) (end 309.502515 99.048499)
-    (stroke (width 0.1) (type default)) (layer "Edge.Cuts"))
-  (gr_circle (center 219.143 73.225) (end 222.893 73.225)
-    (stroke (width 0.1) (type default)) (fill none) (layer "Edge.Cuts"))
-  (gr_arc (start 368.592857 98.048499) (mid 368.299963 98.755606) (end 367.592857 99.048499)
-    (stroke (width 0.1) (type default)) (layer "Edge.Cuts"))
-  (gr_circle (center 141.321 156.653) (end 144.921 156.653)
-    (stroke (width 0.1) (type default)) (fill none) (layer "Edge.Cuts"))
-  (gr_line (start 368.592857 66.1485) (end 368.592857 98.048499)
-    (stroke (width 0.1) (type default)) (layer "Edge.Cuts"))
-  (gr_arc (start 367.592857 65.1485) (mid 368.299963 65.441393) (end 368.592857 66.1485)
-    (stroke (width 0.1) (type default)) (layer "Edge.Cuts"))
-  (gr_circle (center 125.821 143.953) (end 129.420999 143.953)
-    (stroke (width 0.1) (type default)) (fill none) (layer "Edge.Cuts"))
-  (gr_circle (center 169.143 89.851) (end 173.893 89.851)
-    (stroke (width 0.1) (type default)) (fill none) (layer "Edge.Cuts"))
-  (gr_circle (center 147.143 89.851) (end 151.893 89.851)
-    (stroke (width 0.1) (type default)) (fill none) (layer "Edge.Cuts"))
-  (gr_circle (center 141.321 143.953) (end 144.921 143.953)
-    (stroke (width 0.1) (type default)) (fill none) (layer "Edge.Cuts"))
-  (gr_circle (center 191.143 89.851) (end 195.893 89.851)
-    (stroke (width 0.1) (type default)) (fill none) (layer "Edge.Cuts"))
-  (gr_rect (start 307.492857 64.1485) (end 369.592857 103.9985)
-    (stroke (width 0.1) (type default)) (fill none) (layer "F.Fab"))
-  (gr_rect (start 311.042857 67.1585) (end 366.052857 94.6485)
-    (stroke (width 0.1) (type default)) (fill none) (layer "F.Fab"))
-  (gr_text "OLED pixels (active area) 55.01 x 27.49" (at 312.042857 68.5585) (layer "F.Fab")
-    (effects (font (size 1 1) (thickness 0.15)) (justify left))
-  )
-  (gr_text "OLED glass 62.10 x 39.85 -- black past the pixels" (at 308.492857 102.5985) (layer "F.Fab")
-    (effects (font (size 1 1) (thickness 0.15)) (justify left))
-  )
   (segment (start 331.535 159.075) (end 334.075 159.075) (width 0.5) (layer "B.Cu") (net 1))
   (segment (start 328.995 159.075) (end 331.535 159.075) (width 0.5) (layer "B.Cu") (net 1))

Commit message: faceplate: fillet the panel corners, r 6mm
Dylan: a rounder feel. Radius = the wall thickness: the enclosure's outer
corners take the same radius, and at 6 the cavity keeps square inside
corners, so the main board's outline is untouched; any bigger and the
cavity and board would need rounding too. Nothing on the panel comes
within 24mm of a corner. The one cost is screws: at 3mm in, a screw
can no longer sit in the corner, so corner screws go at least 9mm along
the edge (M3 pan head clears the arc by 0.25). Both are generator
checks; none of the screw positions exist yet.

The generator owns it (panel_corner_r_mm, and the panel art's outline).
mkholes.py now draws the whole Edge.Cuts layer from its sources --
outline, holes, OLED window -- replacing mkboard's square gr_rect, and
is idempotent (same 39 items on a second run). panelcheck checks all
four corners are arcs of that radius; it failed on the square board.

Checked: generator --check all pass, placement unchanged; mksch/netcheck
145/145; boardcheck parity 0, clearance 0; DRC --unrouted 0 errors (the
outline closes); panelcheck --strict 14 OK; place.py all 24.
Other:
- outline, holes or cut-outs redrawn
Changed lines of the file:
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@@
     )
   )
+  (gr_circle (center 169.143 89.851) (end 173.893 89.851)
+    (stroke (width 0.1) (type default)) (fill none) (layer "Edge.Cuts"))
+  (gr_circle (center 125.143 73.395) (end 129.893 73.395)
+    (stroke (width 0.1) (type default)) (fill none) (layer "Edge.Cuts"))
+  (gr_circle (center 263.143 89.681) (end 266.893 89.681)
+    (stroke (width 0.1) (type default)) (fill none) (layer "Edge.Cuts"))
+  (gr_circle (center 293.643 89.631) (end 296.443 89.631)
+    (stroke (width 0.1) (type default)) (fill none) (layer "Edge.Cuts"))
+  (gr_circle (center 141.321 156.653) (end 144.921 156.653)
+    (stroke (width 0.1) (type default)) (fill none) (layer "Edge.Cuts"))
+  (gr_circle (center 125.821 169.353) (end 129.420999 169.353)
+    (stroke (width 0.1) (type default)) (fill none) (layer "Edge.Cuts"))
+  (gr_arc (start 106 187.81) (mid 101.757359 186.05264) (end 100 181.81)
+    (stroke (width 0.1) (type default)) (layer "Edge.Cuts"))
+  (gr_line (start 368.592857 66.1485) (end 368.592857 98.048499)
+    (stroke (width 0.1) (type default)) (layer "Edge.Cuts"))
+  (gr_circle (center 241.143 73.225) (end 244.893 73.225)
+    (stroke (width 0.1) (type default)) (fill none) (layer "Edge.Cuts"))
+  (gr_circle (center 133.571 125.453) (end 138.571 125.453)
+    (stroke (width 0.1) (type default)) (fill none) (layer "Edge.Cuts"))
+  (gr_circle (center 147.143 89.851) (end 151.893 89.851)
+    (stroke (width 0.1) (type default)) (fill none) (layer "Edge.Cuts"))
+  (gr_arc (start 100 56) (mid 101.757359 51.757359) (end 106 50)
+    (stroke (width 0.1) (type default)) (layer "Edge.Cuts"))
+  (gr_circle (center 191.143 89.851) (end 195.893 89.851)
+    (stroke (width 0.1) (type default)) (fill none) (layer "Edge.Cuts"))
+  (gr_line (start 308.502515 98.048499) (end 308.502515 66.1485)
+    (stroke (width 0.1) (type default)) (layer "Edge.Cuts"))
+  (gr_circle (center 125.821 156.653) (end 129.420999 156.653)
+    (stroke (width 0.1) (type default)) (fill none) (layer "Edge.Cuts"))
+  (gr_line (start 367.592857 99.048499) (end 309.502515 99.048499)
+    (stroke (width 0.1) (type default)) (layer "Edge.Cuts"))
+  (gr_line (start 106 50) (end 392.285714 50)
+    (stroke (width 0.1) (type default)) (layer "Edge.Cuts"))
+  (gr_line (start 392.285714 187.81) (end 106 187.81)
+    (stroke (width 0.1) (type default)) (layer "Edge.Cuts"))
+  (gr_circle (center 125.821 143.953) (end 129.420999 143.953)
+    (stroke (width 0.1) (type default)) (fill none) (layer "Edge.Cuts"))
+  (gr_arc (start 392.285714 50) (mid 396.528354 51.757359) (end 398.285714 56)
+    (stroke (width 0.1) (type default)) (layer "Edge.Cuts"))
+  (gr_line (start 100 181.81) (end 100 56)
+    (stroke (width 0.1) (type default)) (layer "Edge.Cuts"))
+  (gr_arc (start 368.592857 98.048499) (mid 368.299963 98.755606) (end 367.592857 99.048499)
+    (stroke (width 0.1) (type default)) (layer "Edge.Cuts"))
+  (gr_circle (center 280.643 89.631) (end 283.443 89.631)
+    (stroke (width 0.1) (type default)) (fill none) (layer "Edge.Cuts"))
+  (gr_line (start 398.285714 56) (end 398.285714 181.81)
+    (stroke (width 0.1) (type default)) (layer "Edge.Cuts"))
+  (gr_circle (center 147.143 73.395) (end 151.893 73.395)
+    (stroke (width 0.1) (type default)) (fill none) (layer "Edge.Cuts"))
+  (gr_arc (start 398.285714 181.81) (mid 396.528354 186.05264) (end 392.285714 187.81)
+    (stroke (width 0.1) (type default)) (layer "Edge.Cuts"))
+  (gr_circle (center 219.143 89.681) (end 222.893 89.681)
+    (stroke (width 0.1) (type default)) (fill none) (layer "Edge.Cuts"))
+  (gr_circle (center 125.143 89.851) (end 129.893 89.851)
+    (stroke (width 0.1) (type default)) (fill none) (layer "Edge.Cuts"))
+  (gr_circle (center 191.143 73.395) (end 195.893 73.395)
+    (stroke (width 0.1) (type default)) (fill none) (layer "Edge.Cuts"))
+  (gr_arc (start 367.592857 65.1485) (mid 368.299963 65.441393) (end 368.592857 66.1485)
+    (stroke (width 0.1) (type default)) (layer "Edge.Cuts"))
+  (gr_line (start 309.502515 65.1485) (end 367.592857 65.1485)
+    (stroke (width 0.1) (type default)) (layer "Edge.Cuts"))
+  (gr_circle (center 169.143 73.395) (end 173.893 73.395)
+    (stroke (width 0.1) (type default)) (fill none) (layer "Edge.Cuts"))
+  (gr_circle (center 263.143 73.225) (end 266.893 73.225)
+    (stroke (width 0.1) (type default)) (fill none) (layer "Edge.Cuts"))
+  (gr_circle (center 141.321 143.953) (end 144.921 143.953)
+    (stroke (width 0.1) (type default)) (fill none) (layer "Edge.Cuts"))
   (gr_circle (center 219.143 73.225) (end 222.893 73.225)
     (stroke (width 0.1) (type default)) (fill none) (layer "Edge.Cuts"))
-  (gr_line (start 368.592857 66.1485) (end 368.592857 98.048499)
+  (gr_circle (center 141.321 169.353) (end 144.921 169.353)
+    (stroke (width 0.1) (type default)) (fill none) (layer "Edge.Cuts"))
+  (gr_arc (start 309.502515 99.048499) (mid 308.795409 98.755606) (end 308.502515 98.048499)
+    (stroke (width 0.1) (type default)) (layer "Edge.Cuts"))
+  (gr_arc (start 308.502515 66.1485) (mid 308.795409 65.441393) (end 309.502515 65.1485)
     (stroke (width 0.1) (type default)) (layer "Edge.Cuts"))
   (gr_circle (center 241.143 89.681) (end 244.893 89.681)
     (stroke (width 0.1) (type default)) (fill none) (layer "Edge.Cuts"))
-  (gr_circle (center 125.821 143.953) (end 129.420999 143.953)
-    (stroke (width 0.1) (type default)) (fill none) (layer "Edge.Cuts"))
-  (gr_circle (center 280.643 89.631) (end 283.443 89.631)
-    (stroke (width 0.1) (type default)) (fill none) (layer "Edge.Cuts"))
-  (gr_circle (center 169.143 89.851) (end 173.893 89.851)
-    (stroke (width 0.1) (type default)) (fill none) (layer "Edge.Cuts"))
-  (gr_circle (center 191.143 89.851) (end 195.893 89.851)
-    (stroke (width 0.1) (type default)) (fill none) (layer "Edge.Cuts"))
-  (gr_circle (center 141.321 143.953) (end 144.921 143.953)
-    (stroke (width 0.1) (type default)) (fill none) (layer "Edge.Cuts"))
-  (gr_circle (center 293.643 89.631) (end 296.443 89.631)
-    (stroke (width 0.1) (type default)) (fill none) (layer "Edge.Cuts"))
-  (gr_circle (center 141.321 169.353) (end 144.921 169.353)
-    (stroke (width 0.1) (type default)) (fill none) (layer "Edge.Cuts"))
-  (gr_arc (start 367.592857 65.1485) (mid 368.299963 65.441393) (end 368.592857 66.1485)
-    (stroke (width 0.1) (type default)) (layer "Edge.Cuts"))
-  (gr_circle (center 169.143 73.395) (end 173.893 73.395)
-    (stroke (width 0.1) (type default)) (fill none) (layer "Edge.Cuts"))
-  (gr_circle (center 191.143 73.395) (end 195.893 73.395)
-    (stroke (width 0.1) (type default)) (fill none) (layer "Edge.Cuts"))
-  (gr_circle (center 125.821 169.353) (end 129.420999 169.353)
-    (stroke (width 0.1) (type default)) (fill none) (layer "Edge.Cuts"))
-  (gr_rect (start 100 50) (end 398.285714 187.81)
-    (stroke (width 0.1) (type default)) (fill none) (layer "Edge.Cuts"))
-  (gr_circle (center 125.143 73.395) (end 129.893 73.395)
-    (stroke (width 0.1) (type default)) (fill none) (layer "Edge.Cuts"))
-  (gr_circle (center 241.143 73.225) (end 244.893 73.225)
-    (stroke (width 0.1) (type default)) (fill none) (layer "Edge.Cuts"))
-  (gr_circle (center 263.143 89.681) (end 266.893 89.681)
-    (stroke (width 0.1) (type default)) (fill none) (layer "Edge.Cuts"))
-  (gr_line (start 309.502515 65.1485) (end 367.592857 65.1485)
-    (stroke (width 0.1) (type default)) (layer "Edge.Cuts"))
-  (gr_circle (center 147.143 73.395) (end 151.893 73.395)
-    (stroke (width 0.1) (type default)) (fill none) (layer "Edge.Cuts"))
-  (gr_arc (start 309.502515 99.048499) (mid 308.795409 98.755606) (end 308.502515 98.048499)
-    (stroke (width 0.1) (type default)) (layer "Edge.Cuts"))
-  (gr_arc (start 368.592857 98.048499) (mid 368.299963 98.755606) (end 367.592857 99.048499)
-    (stroke (width 0.1) (type default)) (layer "Edge.Cuts"))
-  (gr_circle (center 125.143 89.851) (end 129.893 89.851)
-    (stroke (width 0.1) (type default)) (fill none) (layer "Edge.Cuts"))
-  (gr_circle (center 125.821 156.653) (end 129.420999 156.653)
-    (stroke (width 0.1) (type default)) (fill none) (layer "Edge.Cuts"))
-  (gr_circle (center 141.321 156.653) (end 144.921 156.653)
-    (stroke (width 0.1) (type default)) (fill none) (layer "Edge.Cuts"))
-  (gr_line (start 308.502515 98.048499) (end 308.502515 66.1485)
-    (stroke (width 0.1) (type default)) (layer "Edge.Cuts"))
-  (gr_circle (center 219.143 89.681) (end 222.893 89.681)
-    (stroke (width 0.1) (type default)) (fill none) (layer "Edge.Cuts"))
-  (gr_circle (center 147.143 89.851) (end 151.893 89.851)
-    (stroke (width 0.1) (type default)) (fill none) (layer "Edge.Cuts"))
-  (gr_arc (start 308.502515 66.1485) (mid 308.795409 65.441393) (end 309.502515 65.1485)
-    (stroke (width 0.1) (type default)) (layer "Edge.Cuts"))
-  (gr_circle (center 133.571 125.453) (end 138.571 125.453)
-    (stroke (width 0.1) (type default)) (fill none) (layer "Edge.Cuts"))
-  (gr_line (start 367.592857 99.048499) (end 309.502515 99.048499)
-    (stroke (width 0.1) (type default)) (layer "Edge.Cuts"))
-  (gr_circle (center 263.143 73.225) (end 266.893 73.225)
-    (stroke (width 0.1) (type default)) (fill none) (layer "Edge.Cuts"))
   (segment (start 331.535 159.075) (end 334.075 159.075) (width 0.5) (layer "B.Cu") (net 1))
