File: hardware/faceplate/vuulgaris-faceplate.kicad_sch (KiCad schematic)
At the start: 54 parts, among them J1 HX JN2.54-2x5P TP H8.9, U1 MSP430FR2675TPT, Y1 32.768kHz FC-135 12.5pF

Commit message: faceplate: pad copper on the board, one open via per bar
The generator drew every bar as its own island -- 800 of them, joined to
nothing. TI's SLAA891 elements are single bodies, so the cross-check turned
into a connectivity decision: one via per bar (Dylan's call), open, not
filled or capped, and open on the back so nothing traps plating chemistry.

Generator: copper() places a 0.3/0.5 via 0.5mm in from each bar's outer
edge; bars too short for one (the 0.197mm slivers, and five thin RX0 bars
behind J1 on pad 4) are bridged along the pad edge to a same-net bar that
has one. Vias walk inward to clear J1's pad rows on the back. Hole and
bridge copper go into the area compensation; --check now measures all four
pads with both counted: 0.00mm worst error (0.72mm and 2.02mm without,
watched failing). 763 vias, 37 bridges.

design/mkpads.py writes SCRUB_PAD_216x10_P1..P4 (bars as roundrect pads
numbered by E's pins, one F.Mask opening, B.Mask open at each via, no
paste, allow_soldermask_bridges) and places E1-E4 and the vias via pcbnew.
panelcheck checks the board's pads and vias against copper() to 1um, and
the generator's keepouts against J1's real pads; both watched failing.

drc.py --unrouted: the board is placed for hand-routing, so unconnected
items are the ratsnest; every other error still fails (watched on a
planted clearance violation). Bare drc.py remains the fab check.

Checked: generator --check all pass, placement file unchanged;
mksch/netcheck 145/145; boardcheck parity 0, clearance 0; DRC --unrouted
0 errors; panelcheck 9 OK; main board DRC 0 errors, place.py all 24.
The other 50 footprints came in from the schematic and are parked off
the outline until the next commit.
Parts:
- E1: footprint (none) -> vuulgaris:SCRUB_PAD_216x10_P1
- E2: footprint (none) -> vuulgaris:SCRUB_PAD_216x10_P2
- E3: footprint (none) -> vuulgaris:SCRUB_PAD_216x10_P3
- E4: footprint (none) -> vuulgaris:SCRUB_PAD_216x10_P4
Changed lines of the file:
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@@
     (property "Reference" "E1" (at 90 348 0) (effects (font (size 1.27 1.27))))
     (property "Value" "scrub pad 1" (at 90 351 0) (effects (font (size 1.27 1.27))))
-    (property "Footprint" "" (at 90 360 0) (effects (font (size 1.27 1.27)) hide))
+    (property "Footprint" "vuulgaris:SCRUB_PAD_216x10_P1" (at 90 360 0) (effects (font (size 1.27 1.27)) hide))
     (property "Datasheet" "" (at 90 360 0) (effects (font (size 1.27 1.27)) hide))
     (pin "1")
@@
     (property "Reference" "E2" (at 90 413 0) (effects (font (size 1.27 1.27))))
     (property "Value" "scrub pad 2" (at 90 416 0) (effects (font (size 1.27 1.27))))
-    (property "Footprint" "" (at 90 425 0) (effects (font (size 1.27 1.27)) hide))
+    (property "Footprint" "vuulgaris:SCRUB_PAD_216x10_P2" (at 90 425 0) (effects (font (size 1.27 1.27)) hide))
     (property "Datasheet" "" (at 90 425 0) (effects (font (size 1.27 1.27)) hide))
     (pin "1")
@@
     (property "Reference" "E3" (at 90 478 0) (effects (font (size 1.27 1.27))))
     (property "Value" "scrub pad 3" (at 90 481 0) (effects (font (size 1.27 1.27))))
-    (property "Footprint" "" (at 90 490 0) (effects (font (size 1.27 1.27)) hide))
+    (property "Footprint" "vuulgaris:SCRUB_PAD_216x10_P3" (at 90 490 0) (effects (font (size 1.27 1.27)) hide))
     (property "Datasheet" "" (at 90 490 0) (effects (font (size 1.27 1.27)) hide))
     (pin "1")
@@
     (property "Reference" "E4" (at 90 543 0) (effects (font (size 1.27 1.27))))
     (property "Value" "scrub pad 4" (at 90 546 0) (effects (font (size 1.27 1.27))))
-    (property "Footprint" "" (at 90 555 0) (effects (font (size 1.27 1.27)) hide))
+    (property "Footprint" "vuulgaris:SCRUB_PAD_216x10_P4" (at 90 555 0) (effects (font (size 1.27 1.27)) hide))
     (property "Datasheet" "" (at 90 555 0) (effects (font (size 1.27 1.27)) hide))
     (pin "1")
